File: EVSE-Easy-Test/EVSE-Easy-Test.sch (KiCad schematic (older format))
At the start: 13 parts, among them J1 Type 2, J2 Conn_01x02, SW1 PP current coding, SW2 CP state coding

Commit message: completed and sent to aisler
Parts:
- J2: value Conn_01x02 -> CP diag
Changed lines of the file:
@@
 P 7900 5150
 F 0 "J2" H 7820 4825 50  0000 C CNN
-F 1 "Conn_01x02" H 7820 4916 50  0000 C CNN
+F 1 "CP diag" H 7820 4916 50  0000 C CNN
 F 2 "Pin_Headers:Pin_Header_Straight_1x02_Pitch2.54mm" H 7900 5150 50  0001 C CNN
 F 3 "~" H 7900 5150 50  0001 C CNN

Commit message: second prototype as ordered
Parts:
- D1: footprint Diodes_THT:D_DO-41_SOD81_P7.62mm_Horizontal -> local:D_DO-41_SOD81_P7.62mm_Horizontal
- J1: footprint local:Type2-Solderpads -> local:RIACon175_3poles_AKL175-03; Reichelt Artikelnummer (none) -> AKL 175-03
- J2: footprint Pin_Headers:Pin_Header_Straight_1x02_Pitch2.54mm -> local:Pin_Header_Straight_1x02_Pitch2.54mm
- R1, R2, R3, R4, R5, R6, R7, R8: footprint Resistors_THT:R_Axial_DIN0204_L3.6mm_D1.6mm_P7.62mm_Horizontal -> local:R_Axial_DIN0204_L3.6mm_D1.6mm_P7.62mm_Horizontal
Connections:
- net PE: now also R6.1, SW2.6; no longer SW2.12, SW2.5, SW2.8
- net at D1.1 (K), SW2.3, SW2.4: now also SW2.5; no longer SW2.2
- net at D1.2 (A), R6.2: now also SW2.1, SW2.14; no longer SW2.6
- net at SW2.10: now also R7.2, SW2.7; no longer R3.2
- net at SW2.11: now also R3.2
- net at SW2.9: no longer R7.2
- no-connect marks 11 -> 12
Other:
- note added: "Control Pilot states:\n1: Diode fault (in state C)\n2: A - vehicle disconnected\n3: B - vehicle ready\n4: C - vehicle requested charging\n5: D - vehicle requested vented charging\n6: E - CP-PE short, cable or vehicle failure\n"
- note removed: "Control Pilot states:\n1: A - vehicle disconnected\n2: B - vehicle ready\n3: C - vehicle requested charging\n4: D - vehicle requested vented charging\n5: E - CP-PE short, cable or vehicle failure\n6: Diode fault"
- moved on the sheet: D1, R3, R6, R7, SW2
Changed lines of the file:
@@
 L pspice:DIODE D1
 U 1 1 5C013AD5
-P 3150 5150
-F 0 "D1" H 3150 5415 50  0000 C CNN
-F 1 "1N4007" H 3150 5324 50  0000 C CNN
-F 2 "Diodes_THT:D_DO-41_SOD81_P7.62mm_Horizontal" H 3150 5150 50  0001 C CNN
-F 3 "~" H 3150 5150 50  0001 C CNN
-	1    3150 5150
+P 3150 5200
+F 0 "D1" H 3150 5465 50  0000 C CNN
+F 1 "1N4007" H 3150 5374 50  0000 C CNN
+F 2 "local:D_DO-41_SOD81_P7.62mm_Horizontal" H 3150 5200 50  0001 C CNN
+F 3 "~" H 3150 5200 50  0001 C CNN
+	1    3150 5200
 	1    0    0    -1
 $EndComp
@@
 L Device:R R6
 U 1 1 5C013C45
-P 3650 5150
-F 0 "R6" V 3443 5150 50  0000 C CNN
-F 1 "2k7" V 3534 5150 50  0000 C CNN
-F 2 "Resistors_THT:R_Axial_DIN0204_L3.6mm_D1.6mm_P7.62mm_Horizontal" V 3580 5150 50  0001 C CNN
-F 3 "~" H 3650 5150 50  0001 C CNN
-	1    3650 5150
+P 3650 5200
+F 0 "R6" V 3443 5200 50  0000 C CNN
+F 1 "2k7" V 3534 5200 50  0000 C CNN
+F 2 "local:R_Axial_DIN0204_L3.6mm_D1.6mm_P7.62mm_Horizontal" V 3580 5200 50  0001 C CNN
+F 3 "~" H 3650 5200 50  0001 C CNN
+	1    3650 5200
 	0    1    1    0
 $EndComp
@@
 F 0 "J2" H 7820 4825 50  0000 C CNN
 F 1 "CP diag" H 7820 4916 50  0000 C CNN
-F 2 "Pin_Headers:Pin_Header_Straight_1x02_Pitch2.54mm" H 7900 5150 50  0001 C CNN
+F 2 "local:Pin_Header_Straight_1x02_Pitch2.54mm" H 7900 5150 50  0001 C CNN
 F 3 "~" H 7900 5150 50  0001 C CNN
 	1    7900 5150
@@
 F 0 "J1" H 7670 1775 50  0000 C CNN
 F 1 "Type 2" H 7670 1866 50  0000 C CNN
-F 2 "local:Type2-Solderpads" H 7750 2100 50  0001 C CNN
-F 3 "~" H 7750 2100 50  0001 C CNN
+F 2 "local:RIACon175_3poles_AKL175-03" H 7750 2100 50  0001 C CNN
+F 3 "https://cdn-reichelt.de/documents/datenblatt/D700/AKL_175-03.PDF" H 7750 2100 50  0001 C CNN
+F 4 "AKL 175-03" H 7750 2100 50  0001 C CNN "Reichelt Artikelnummer"
 	1    7750 2100
 	-1   0    0    1
@@
 L Switch:SW_Rotary2x6 SW2
 U 1 1 5C014C66
-P 1850 5550
-F 0 "SW2" H 1900 6328 50  0000 C CNN
-F 1 "CP state coding" H 1900 6237 50  0000 C CNN
-F 2 "local:LorlinCK-1060" H 1750 6150 50  0001 C CNN
-F 3 "http://cdn-reichelt.de/documents/datenblatt/C200/DS-Serie%23LOR.pdf" H 1750 6150 50  0001 C CNN
-	1    1850 5550
+P 1850 5500
+F 0 "SW2" H 1900 6278 50  0000 C CNN
+F 1 "CP state coding" H 1900 6187 50  0000 C CNN
+F 2 "local:LorlinCK-1060" H 1750 6100 50  0001 C CNN
+F 3 "http://cdn-reichelt.de/documents/datenblatt/C200/DS-Serie%23LOR.pdf" H 1750 6100 50  0001 C CNN
+	1    1850 5500
 	1    0    0    -1
 $EndComp
@@
 F 0 "R2" H 2830 2404 50  0000 R CNN
 F 1 "100" H 2830 2495 50  0000 R CNN
-F 2 "Resistors_THT:R_Axial_DIN0204_L3.6mm_D1.6mm_P7.62mm_Horizontal" V 2830 2450 50  0001 C CNN
+F 2 "local:R_Axial_DIN0204_L3.6mm_D1.6mm_P7.62mm_Horizontal" V 2830 2450 50  0001 C CNN
 F 3 "~" H 2900 2450 50  0001 C CNN
 	1    2900 2450
@@
 F 0 "R4" H 3130 2404 50  0000 R CNN
 F 1 "220" H 3130 2495 50  0000 R CNN
-F 2 "Resistors_THT:R_Axial_DIN0204_L3.6mm_D1.6mm_P7.62mm_Horizontal" V 3130 2450 50  0001 C CNN
+F 2 "local:R_Axial_DIN0204_L3.6mm_D1.6mm_P7.62mm_Horizontal" V 3130 2450 50  0001 C CNN
 F 3 "~" H 3200 2450 50  0001 C CNN
 	1    3200 2450
@@
 F 0 "R5" H 3430 2404 50  0000 R CNN
 F 1 "680" H 3430 2495 50  0000 R CNN
-F 2 "Resistors_THT:R_Axial_DIN0204_L3.6mm_D1.6mm_P7.62mm_Horizontal" V 3430 2450 50  0001 C CNN
+F 2 "local:R_Axial_DIN0204_L3.6mm_D1.6mm_P7.62mm_Horizontal" V 3430 2450 50  0001 C CNN
 F 3 "~" H 3500 2450 50  0001 C CNN
 	1    3500 2450
@@
 F 0 "R8" H 3730 2404 50  0000 R CNN
 F 1 "1k5" H 3730 2495 50  0000 R CNN
-F 2 "Resistors_THT:R_Axial_DIN0204_L3.6mm_D1.6mm_P7.62mm_Horizontal" V 3730 2450 50  0001 C CNN
+F 2 "local:R_Axial_DIN0204_L3.6mm_D1.6mm_P7.62mm_Horizontal" V 3730 2450 50  0001 C CNN
 F 3 "~" H 3800 2450 50  0001 C CNN
 	1    3800 2450
@@
 F 0 "R1" H 2530 2404 50  0000 R CNN
 F 1 "3k3" H 2530 2495 50  0000 R CNN
-F 2 "Resistors_THT:R_Axial_DIN0204_L3.6mm_D1.6mm_P7.62mm_Horizontal" V 2530 2450 50  0001 C CNN
+F 2 "local:R_Axial_DIN0204_L3.6mm_D1.6mm_P7.62mm_Horizontal" V 2530 2450 50  0001 C CNN
 F 3 "~" H 2600 2450 50  0001 C CNN
 	1    2600 2450
@@
 Text Notes 2900 3500 0    50   ~ 0
 Current coding:\n1: not connected\n2: 13A\n3: 20A\n4: 32A\n5: 63A\n6: Invalid coding
-Text GLabel 1150 5250 0    50   Input ~ 0
+Text GLabel 1150 5200 0    50   Input ~ 0
 CP
 Wire Wire Line
-	1100 5250 1450 5250
-NoConn ~ 2350 4950
-Wire Wire Line
-	2350 5050 2700 5050
-Wire Wire Line
-	2700 5050 2700 5150
-Wire Wire Line
-	2700 5150 2950 5150
-Wire Wire Line
-	2350 5150 2700 5150
-Connection ~ 2700 5150
-Wire Wire Line
-	2350 5250 2700 5250
-Wire Wire Line
-	2700 5250 2700 5150
-Wire Wire Line
-	3350 5150 3400 5150
-Wire Wire Line
-	3800 5150 4000 5150
-Wire Wire Line
-	4000 5150 4000 5550
-Wire Wire Line
-	4000 5550 1350 5550
-Wire Wire Line
-	1350 5550 1350 5950
-Wire Wire Line
-	1350 5950 1450 5950
+	1100 5200 1450 5200
+NoConn ~ 2350 5000
+Wire Wire Line
+	2350 5100 2700 5100
+Wire Wire Line
+	2700 5100 2700 5200
+Wire Wire Line
+	2700 5200 2950 5200
+Wire Wire Line
+	2350 5200 2700 5200
+Connection ~ 2700 5200
+Wire Wire Line
+	2350 5300 2700 5300
+Wire Wire Line
+	2700 5300 2700 5200
+Wire Wire Line
+	3800 5200 4000 5200
 Text Notes 2950 6950 0    50   ~ 0
-Control Pilot states:\n1: A - vehicle disconnected\n2: B - vehicle ready\n3: C - vehicle requested charging\n4: D - vehicle requested vented charging\n5: E - CP-PE short, cable or vehicle failure\n6: Diode fault
-Wire Wire Line
-	2350 5450 3400 5450
-Wire Wire Line
-	3400 5450 3400 5150
-Connection ~ 3400 5150
-Wire Wire Line
-	3400 5150 3500 5150
-NoConn ~ 2350 5650
-Text GLabel 4300 6150 2    50   Input ~ 0
+Control Pilot states:\n1: Diode fault (in state C)\n2: A - vehicle disconnected\n3: B - vehicle ready\n4: C - vehicle requested charging\n5: D - vehicle requested vented charging\n6: E - CP-PE short, cable or vehicle failure\n
+NoConn ~ 2350 5700
+Text GLabel 4300 6200 2    50   Input ~ 0
 PE
-Wire Wire Line
-	2350 5750 4000 5750
-Wire Wire Line
-	4000 5750 4000 5850
 $Comp
 L Device:R R7
 U 1 1 5C01E965
-P 3650 5850
-F 0 "R7" V 3600 6050 50  0000 C CNN
-F 1 "1k2" V 3700 6050 50  0000 C CNN
-F 2 "Resistors_THT:R_Axial_DIN0204_L3.6mm_D1.6mm_P7.62mm_Horizontal" V 3580 5850 50  0001 C CNN
-F 3 "~" H 3650 5850 50  0001 C CNN
-	1    3650 5850
+P 3650 5900
+F 0 "R7" V 3600 6100 50  0000 C CNN
+F 1 "1k2" V 3700 6100 50  0000 C CNN
+F 2 "local:R_Axial_DIN0204_L3.6mm_D1.6mm_P7.62mm_Horizontal" V 3580 5900 50  0001 C CNN
+F 3 "~" H 3650 5900 50  0001 C CNN
+	1    3650 5900
 	0    1    1    0
 $EndComp
 Wire Wire Line
-	2350 5850 3500 5850
-Wire Wire Line
-	3800 5850 4000 5850
-Connection ~ 4000 5850
+	3800 5900 4000 5900
+Connection ~ 4000 5900
 $Comp
 L Device:R R3
 U 1 1 5C0200DE
-P 2900 5950
-F 0 "R3" V 2850 6150 50  0000 C CNN
-F 1 "270" V 2950 6150 50  0000 C CNN
-F 2 "Resistors_THT:R_Axial_DIN0204_L3.6mm_D1.6mm_P7.62mm_Horizontal" V 2830 5950 50  0001 C CNN
-F 3 "~" H 2900 5950 50  0001 C CNN
-	1    2900 5950
+P 3150 6000
+F 0 "R3" V 3100 6200 50  0000 C CNN
+F 1 "270" V 3200 6200 50  0000 C CNN
+F 2 "local:R_Axial_DIN0204_L3.6mm_D1.6mm_P7.62mm_Horizontal" V 3080 6000 50  0001 C CNN
+F 3 "~" H 3150 6000 50  0001 C CNN
+	1    3150 6000
 	0    1    1    0
 $EndComp
-Wire Wire Line
-	2350 5350 4150 5350
-NoConn ~ 2350 6050
-Wire Wire Line
-	2350 6150 4000 6150
-Wire Wire Line
-	4000 6150 4000 5950
-Connection ~ 4000 5950
-Wire Wire Line
-	4000 5850 4000 5950
-Wire Wire Line
-	4000 6150 4150 6150
-Connection ~ 4000 6150
-Wire Wire Line
-	4150 5350 4150 6150
-Connection ~ 4150 6150
-Wire Wire Line
-	4150 6150 4300 6150
-Wire Wire Line
-	2350 5950 2750 5950
-Wire Wire Line
-	3050 5950 4000 5950
+NoConn ~ 2350 6100
 Text Notes 7300 1350 0    118  ~ 24
 Type 2 plug connector
@@
 Wire Wire Line
 	8100 5150 8250 5150
+Wire Wire Line
+	4000 5200 4000 5400
+NoConn ~ 2350 5800
+Wire Wire Line
+	4000 5900 4000 6000
+Wire Wire Line
+	2350 6000 3000 6000
+Wire Wire Line
+	3300 6000 4000 6000
+Connection ~ 4000 6000
+Wire Wire Line
+	4000 6000 4000 6200
+Wire Wire Line
+	1450 5900 1450 5500
+Wire Wire Line
+	4000 6200 4300 6200
+Wire Wire Line
+	2350 5400 4000 5400
+Connection ~ 4000 5400
+Wire Wire Line
+	4000 5400 4000 5900
+Wire Wire Line
+	2350 5900 3450 5900
+Wire Wire Line
+	3450 5600 3450 5900
+Wire Wire Line
+	2350 5600 3450 5600
+Connection ~ 3450 5900
+Wire Wire Line
+	3450 5900 3500 5900
+Wire Wire Line
+	3350 5200 3450 5200
+Wire Wire Line
+	3450 5200 3450 5500
+Wire Wire Line
+	1450 5500 3450 5500
+Connection ~ 3450 5200
+Wire Wire Line
+	3450 5200 3500 5200
+Wire Wire Line
+	3450 5200 3450 4900
+Wire Wire Line
+	2350 4900 3450 4900
 $EndSCHEMATC
